File: Rev_0.2/SaturnDin/MegaAV_Saturn_rev0.2.kicad_sch (KiCad schematic)
At the start: 150 parts, among them CN1 MD-90SM_MD2, P1 SMD_Conn_01x01, U1 ICS501, U2 MC33204, U3 THS7374, U4 MC33204, U5 AD725

Commit message: Add files via upload
Parts:
- C30, C31: value 5600p -> 1800p
Changed lines of the file:
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@@
 			)
 		)
-		(property "Value" "5600p"
+		(property "Value" "1800p"
 			(at 265.938 113.538 90)
 			(effects
@@
 			)
 		)
-		(property "Value" "5600p"
+		(property "Value" "1800p"
 			(at 265.938 179.578 90)
 			(effects
