File: VA1_Beta/MegaAV_VA1.kicad_sch (KiCad schematic)
At the start: 176 parts, among them CN1 MD-90SM_MD2, P1 SMD_Conn_01x01, U1 4070, U2 74HCT123, U3 TS924, U4 THS7374, U5 ICS501, U6 TS922, U7 TS924, U8 AD723

Commit message: erc
Parts:
- R59, R6: symbol 3bpV2A_RevC-eagle-import:R-US_R0603 -> Device:R_US
- Z1: symbol Connector:Conn_01x33_Pin -> Connector_Generic_MountingPin:Conn_01x33_MountingPin
Connections:
- no-connect marks 0 -> 4
Other:
- moved on the sheet: C37, C40, C49, C50, D2, L1, R50, R51, U1C
