File: VA1_Beta/MegaAV_VA1.kicad_sch (KiCad schematic)
At the start: 176 parts, among them CN1 MD-90SM_MD2, P1 SMD_Conn_01x01, U1 4070, U2 74HCT123, U3 TS924, U4 THS7374, U5 ICS501, U6 TS922, U7 TS924, U8 AD723

Commit message: Fix ERC
Parts:
- J1: renamed from Z1; value Conn_01x33_Pin -> Conn_01x33_MountingPin; footprint Connector_FFC-FPC:Molex_502244-3330_1x33-1MP_P0.5mm_Horizontal -> (none); symbol Connector:Conn_01x33_Pin -> Connector_Generic_MountingPin:Conn_01x33_MountingPin
Connections:
- no-connect marks 0 -> 4
Other:
- company: Developed By: Ace9921, RIP-Felix, RGBeter, Villahed94 -> Developed By: RIP-Felix, RGBeter, Villahed94
- moved on the sheet: C40, C49, C50, D2, L1, R59, U1C
