File: VA1_Beta/MegaAV_VA1.kicad_pcb (KiCad board)
At the start: 4 copper layers, 50 x 50 mm, 177 parts, among them CN1 MD-90SM_MD2, P1 SMD_Conn_01x01, U1 4070, U2 74HCT123, U3 TS924, U4 THS7374, U5 ICS501, U6 TS922, U7 TS924, U8 AD723

Commit message: Deal with DRC
Routing:
- net GND: track 56.3 -> 66.6 mm, vias 76 -> 77
- net +5V: track 270.3 -> 268.9 mm
- net /B-IN: track 6.09 -> 5.33 mm
- net /32X_L: track 44.2 -> 43.5 mm
- net /STDSEL: track 19.9 -> 19.2 mm
- net Net-(FMR_2-B): track 2.28 -> 1.65 mm
- net Net-(C24-Pad2): track 4.70 -> 4.08 mm
- net /CD_L: track 63.0 -> 62.4 mm
Other:
- board size 50 x 50 mm -> 49.9 x 50 mm
